File: iSpindel/deska.sch (EAGLE design)
At the start: 14 parts

Commit message: zmeny desky
Connections:
- net +5V: now also OUT+.1
- net GND: now also OUT-.1
Other:
- moved on the sheet: JP1, JP3
Changed lines of the file:
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@@
 <grid distance="0.1" unitdist="inch" unit="inch" style="lines" multiple="1" display="no" altdistance="0.01" altunitdist="inch" altunit="inch"/>
 <layers>
-<layer number="1" name="Top" color="4" fill="1" visible="no" active="no"/>
-<layer number="16" name="Bottom" color="1" fill="1" visible="no" active="no"/>
-<layer number="17" name="Pads" color="2" fill="1" visible="no" active="no"/>
-<layer number="18" name="Vias" color="2" fill="1" visible="no" active="no"/>
-<layer number="19" name="Unrouted" color="6" fill="1" visible="no" active="no"/>
-<layer number="20" name="Dimension" color="15" fill="1" visible="no" active="no"/>
-<layer number="21" name="tPlace" color="7" fill="1" visible="no" active="no"/>
-<layer number="22" name="bPlace" color="7" fill="1" visible="no" active="no"/>
-<layer number="23" name="tOrigins" color="15" fill="1" visible="no" active="no"/>
-<layer number="24" name="bOrigins" color="15" fill="1" visible="no" active="no"/>
-<layer number="25" name="tNames" color="7" fill="1" visible="no" active="no"/>
-<layer number="26" name="bNames" color="7" fill="1" visible="no" active="no"/>
-<layer number="27" name="tValues" color="7" fill="1" visible="no" active="no"/>
-<layer number="28" name="bValues" color="7" fill="1" visible="no" active="no"/>
+<layer number="1" name="Top" color="4" fill="1" visible="yes" active="no"/>
+<layer number="16" name="Bottom" color="1" fill="1" visible="yes" active="no"/>
+<layer number="17" name="Pads" color="2" fill="1" visible="yes" active="no"/>
+<layer number="18" name="Vias" color="2" fill="1" visible="yes" active="no"/>
+<layer number="19" name="Unrouted" color="6" fill="1" visible="yes" active="no"/>
+<layer number="20" name="Dimension" color="15" fill="1" visible="yes" active="no"/>
+<layer number="21" name="tPlace" color="7" fill="1" visible="yes" active="no"/>
+<layer number="22" name="bPlace" color="7" fill="1" visible="yes" active="no"/>
+<layer number="23" name="tOrigins" color="15" fill="1" visible="yes" active="no"/>
+<layer number="24" name="bOrigins" color="15" fill="1" visible="yes" active="no"/>
+<layer number="25" name="tNames" color="7" fill="1" visible="yes" active="no"/>
+<layer number="26" name="bNames" color="7" fill="1" visible="yes" active="no"/>
+<layer number="27" name="tValues" color="7" fill="1" visible="yes" active="no"/>
+<layer number="28" name="bValues" color="7" fill="1" visible="yes" active="no"/>
 <layer number="29" name="tStop" color="7" fill="3" visible="no" active="no"/>
 <layer number="30" name="bStop" color="7" fill="6" visible="no" active="no"/>
@@
 <layer number="35" name="tGlue" color="7" fill="4" visible="no" active="no"/>
 <layer number="36" name="bGlue" color="7" fill="5" visible="no" active="no"/>
-<layer number="37" name="tTest" color="7" fill="1" visible="no" active="no"/>
-<layer number="38" name="bTest" color="7" fill="1" visible="no" active="no"/>
+<layer number="37" name="tTest" color="7" fill="1" visible="yes" active="no"/>
+<layer number="38" name="bTest" color="7" fill="1" visible="yes" active="no"/>
 <layer number="39" name="tKeepout" color="4" fill="11" visible="no" active="no"/>
 <layer number="40" name="bKeepout" color="1" fill="11" visible="no" active="no"/>
@@
 <layer number="44" name="Drills" color="7" fill="1" visible="no" active="no"/>
 <layer number="45" name="Holes" color="7" fill="1" visible="no" active="no"/>
-<layer number="46" name="Milling" color="3" fill="1" visible="no" active="no"/>
-<layer number="47" name="Measures" color="7" fill="1" visible="no" active="no"/>
-<layer number="48" name="Document" color="7" fill="1" visible="no" active="no"/>
-<layer number="49" name="Reference" color="7" fill="1" visible="no" active="no"/>
-<layer number="51" name="tDocu" color="7" fill="1" visible="no" active="no"/>
-<layer number="52" name="bDocu" color="7" fill="1" visible="no" active="no"/>
+<layer number="46" name="Milling" color="3" fill="1" visible="yes" active="no"/>
+<layer number="47" name="Measures" color="7" fill="1" visible="yes" active="no"/>
+<layer number="48" name="Document" color="7" fill="1" visible="yes" active="no"/>
+<layer number="49" name="Reference" color="7" fill="1" visible="yes" active="no"/>
+<layer number="51" name="tDocu" color="7" fill="1" visible="yes" active="no"/>
+<layer number="52" name="bDocu" color="7" fill="1" visible="yes" active="no"/>
 <layer number="90" name="Modules" color="5" fill="1" visible="yes" active="yes"/>
 <layer number="91" name="Nets" color="2" fill="1" visible="yes" active="yes"/>
@@
 <part name="BAT-1" library="pinhead" deviceset="PINHD-1X1" device=""/>
 <part name="BAT+1" library="pinhead" deviceset="PINHD-1X1" device=""/>
+<part name="P+2" library="supply1" deviceset="+5V" device=""/>
+<part name="GND2" library="supply1" deviceset="GND" device=""/>
 </parts>
 <sheets>
@@
 <instance part="BAT+" gate="G$1" x="43.18" y="58.42"/>
 <instance part="BAT-" gate="G$1" x="43.18" y="50.8"/>
-<instance part="JP1" gate="A" x="81.28" y="45.72" rot="R90"/>
-<instance part="JP3" gate="A" x="78.74" y="58.42" rot="R270"/>
+<instance part="JP1" gate="A" x="81.28" y="50.8" rot="R90"/>
+<instance part="JP3" gate="A" x="78.74" y="55.88" rot="R270"/>
 <instance part="+3V1" gate="G$1" x="71.12" y="73.66"/>
-<instance part="P+1" gate="1" x="71.12" y="30.48" rot="R180"/>
+<instance part="P+1" gate="1" x="71.12" y="35.56" rot="R180"/>
 <instance part="GND1" gate="1" x="73.66" y="25.4"/>
 <instance part="DS18B20" gate="A" x="109.22" y="78.74" rot="R90"/>
@@
 <instance part="BAT-1" gate="G$1" x="58.42" y="50.8"/>
 <instance part="BAT+1" gate="G$1" x="58.42" y="58.42"/>
+<instance part="P+2" gate="1" x="48.26" y="73.66"/>
+<instance part="GND2" gate="1" x="40.64" y="33.02"/>
 </instances>
 <busses>
@@
 <pinref part="JP3" gate="A" pin="8"/>
 <pinref part="+3V1" gate="G$1" pin="+3V3"/>
-<wire x1="71.12" y1="60.96" x2="71.12" y2="68.58" width="0.1524" layer="91"/>
+<wire x1="71.12" y1="58.42" x2="71.12" y2="68.58" width="0.1524" layer="91"/>
 <pinref part="DS18B20" gate="A" pin="1"/>
 <wire x1="71.12" y1="68.58" x2="71.12" y2="71.12" width="0.1524" layer="91"/>
@@
 <pinref part="JP1" gate="A" pin="1"/>
 <pinref part="P+1" gate="1" pin="+5V"/>
-<wire x1="71.12" y1="43.18" x2="71.12" y2="38.1" width="0.1524" layer="91"/>
-<wire x1="71.12" y1="38.1" x2="71.12" y2="33.02" width="0.1524" layer="91"/>
-<wire x1="43.18" y1="66.04" x2="63.5" y2="66.04" width="0.1524" layer="91"/>
-<wire x1="63.5" y1="66.04" x2="63.5" y2="38.1" width="0.1524" layer="91"/>
-<wire x1="63.5" y1="38.1" x2="71.12" y2="38.1" width="0.1524" layer="91"/>
-<junction x="71.12" y="38.1"/>
+<wire x1="71.12" y1="48.26" x2="71.12" y2="38.1" width="0.1524" layer="91"/>
+</segment>
+<segment>
+<pinref part="OUT+" gate="G$1" pin="1"/>
+<wire x1="40.64" y1="66.04" x2="40.64" y2="71.12" width="0.1524" layer="91"/>
+<pinref part="P+2" gate="1" pin="+5V"/>
+<wire x1="40.64" y1="71.12" x2="48.26" y2="71.12" width="0.1524" layer="91"/>
 </segment>
 </net>
@@
 <pinref part="JP1" gate="A" pin="2"/>
 <pinref part="GND1" gate="1" pin="GND"/>
-<wire x1="73.66" y1="43.18" x2="73.66" y2="35.56" width="0.1524" layer="91"/>
-<wire x1="73.66" y1="35.56" x2="73.66" y2="27.94" width="0.1524" layer="91"/>
-<wire x1="73.66" y1="35.56" x2="111.76" y2="35.56" width="0.1524" layer="91"/>
-<junction x="73.66" y="35.56"/>
+<wire x1="73.66" y1="48.26" x2="73.66" y2="40.64" width="0.1524" layer="91"/>
+<wire x1="73.66" y1="40.64" x2="73.66" y2="27.94" width="0.1524" layer="91"/>
+<wire x1="73.66" y1="40.64" x2="111.76" y2="40.64" width="0.1524" layer="91"/>
+<junction x="73.66" y="40.64"/>
 <pinref part="DS18B20" gate="A" pin="3"/>
-<wire x1="111.76" y1="76.2" x2="111.76" y2="35.56" width="0.1524" layer="91"/>
-<wire x1="43.18" y1="43.18" x2="48.26" y2="43.18" width="0.1524" layer="91"/>
-<wire x1="48.26" y1="43.18" x2="48.26" y2="27.94" width="0.1524" layer="91"/>
-<wire x1="48.26" y1="27.94" x2="73.66" y2="27.94" width="0.1524" layer="91"/>
-<junction x="73.66" y="27.94"/>
+<wire x1="111.76" y1="76.2" x2="111.76" y2="40.64" width="0.1524" layer="91"/>
+</segment>
+<segment>
+<pinref part="GND2" gate="1" pin="GND"/>
+<pinref part="OUT-" gate="G$1" pin="1"/>
+<wire x1="40.64" y1="35.56" x2="40.64" y2="43.18" width="0.1524" layer="91"/>
 </segment>
 </net>
@@
 <pinref part="JP3" gate="A" pin="2"/>
 <pinref part="R2" gate="G$1" pin="2"/>
-<wire x1="86.36" y1="60.96" x2="86.36" y2="73.66" width="0.1524" layer="91"/>
+<wire x1="86.36" y1="58.42" x2="86.36" y2="73.66" width="0.1524" layer="91"/>
 </segment>
 </net>
@@
 <segment>
 <pinref part="JP3" gate="A" pin="1"/>
-<wire x1="88.9" y1="60.96" x2="88.9" y2="76.2" width="0.1524" layer="91"/>
+<wire x1="88.9" y1="58.42" x2="88.9" y2="76.2" width="0.1524" layer="91"/>
 <pinref part="R3" gate="G$1" pin="2"/>
 <wire x1="88.9" y1="76.2" x2="91.44" y2="76.2" width="0.1524" layer="91"/>
@@
 <segment>
 <pinref part="JP3" gate="A" pin="3"/>
-<wire x1="83.82" y1="60.96" x2="83.82" y2="71.12" width="0.1524" layer="91"/>
+<wire x1="83.82" y1="58.42" x2="83.82" y2="71.12" width="0.1524" layer="91"/>
 <pinref part="R3" gate="G$1" pin="1"/>
 <wire x1="81.28" y1="78.74" x2="81.28" y2="71.12" width="0.1524" layer="91"/>

Commit message: deska
Parts:
- added IN+1, IN-1: (no value), pinhead:PINHD-1X1
Changed lines of the file:
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@@
 <grid distance="0.1" unitdist="inch" unit="inch" style="lines" multiple="1" display="no" altdistance="0.01" altunitdist="inch" altunit="inch"/>
 <layers>
-<layer number="1" name="Top" color="4" fill="1" visible="yes" active="no"/>
-<layer number="16" name="Bottom" color="1" fill="1" visible="yes" active="no"/>
-<layer number="17" name="Pads" color="2" fill="1" visible="yes" active="no"/>
-<layer number="18" name="Vias" color="2" fill="1" visible="yes" active="no"/>
-<layer number="19" name="Unrouted" color="6" fill="1" visible="yes" active="no"/>
-<layer number="20" name="Dimension" color="15" fill="1" visible="yes" active="no"/>
-<layer number="21" name="tPlace" color="7" fill="1" visible="yes" active="no"/>
-<layer number="22" name="bPlace" color="7" fill="1" visible="yes" active="no"/>
-<layer number="23" name="tOrigins" color="15" fill="1" visible="yes" active="no"/>
-<layer number="24" name="bOrigins" color="15" fill="1" visible="yes" active="no"/>
-<layer number="25" name="tNames" color="7" fill="1" visible="yes" active="no"/>
-<layer number="26" name="bNames" color="7" fill="1" visible="yes" active="no"/>
-<layer number="27" name="tValues" color="7" fill="1" visible="yes" active="no"/>
-<layer number="28" name="bValues" color="7" fill="1" visible="yes" active="no"/>
+<layer number="1" name="Top" color="4" fill="1" visible="no" active="no"/>
+<layer number="16" name="Bottom" color="1" fill="1" visible="no" active="no"/>
+<layer number="17" name="Pads" color="2" fill="1" visible="no" active="no"/>
+<layer number="18" name="Vias" color="2" fill="1" visible="no" active="no"/>
+<layer number="19" name="Unrouted" color="6" fill="1" visible="no" active="no"/>
+<layer number="20" name="Dimension" color="15" fill="1" visible="no" active="no"/>
+<layer number="21" name="tPlace" color="7" fill="1" visible="no" active="no"/>
+<layer number="22" name="bPlace" color="7" fill="1" visible="no" active="no"/>
+<layer number="23" name="tOrigins" color="15" fill="1" visible="no" active="no"/>
+<layer number="24" name="bOrigins" color="15" fill="1" visible="no" active="no"/>
+<layer number="25" name="tNames" color="7" fill="1" visible="no" active="no"/>
+<layer number="26" name="bNames" color="7" fill="1" visible="no" active="no"/>
+<layer number="27" name="tValues" color="7" fill="1" visible="no" active="no"/>
+<layer number="28" name="bValues" color="7" fill="1" visible="no" active="no"/>
 <layer number="29" name="tStop" color="7" fill="3" visible="no" active="no"/>
 <layer number="30" name="bStop" color="7" fill="6" visible="no" active="no"/>
@@
 <layer number="35" name="tGlue" color="7" fill="4" visible="no" active="no"/>
 <layer number="36" name="bGlue" color="7" fill="5" visible="no" active="no"/>
-<layer number="37" name="tTest" color="7" fill="1" visible="yes" active="no"/>
-<layer number="38" name="bTest" color="7" fill="1" visible="yes" active="no"/>
+<layer number="37" name="tTest" color="7" fill="1" visible="no" active="no"/>
+<layer number="38" name="bTest" color="7" fill="1" visible="no" active="no"/>
 <layer number="39" name="tKeepout" color="4" fill="11" visible="no" active="no"/>
 <layer number="40" name="bKeepout" color="1" fill="11" visible="no" active="no"/>
@@
 <layer number="44" name="Drills" color="7" fill="1" visible="no" active="no"/>
 <layer number="45" name="Holes" color="7" fill="1" visible="no" active="no"/>
-<layer number="46" name="Milling" color="3" fill="1" visible="yes" active="no"/>
-<layer number="47" name="Measures" color="7" fill="1" visible="yes" active="no"/>
-<layer number="48" name="Document" color="7" fill="1" visible="yes" active="no"/>
-<layer number="49" name="Reference" color="7" fill="1" visible="yes" active="no"/>
-<layer number="51" name="tDocu" color="7" fill="1" visible="yes" active="no"/>
-<layer number="52" name="bDocu" color="7" fill="1" visible="yes" active="no"/>
+<layer number="46" name="Milling" color="3" fill="1" visible="no" active="no"/>
+<layer number="47" name="Measures" color="7" fill="1" visible="no" active="no"/>
+<layer number="48" name="Document" color="7" fill="1" visible="no" active="no"/>
+<layer number="49" name="Reference" color="7" fill="1" visible="no" active="no"/>
+<layer number="51" name="tDocu" color="7" fill="1" visible="no" active="no"/>
+<layer number="52" name="bDocu" color="7" fill="1" visible="no" active="no"/>
 <layer number="90" name="Modules" color="5" fill="1" visible="yes" active="yes"/>
 <layer number="91" name="Nets" color="2" fill="1" visible="yes" active="yes"/>
@@
 <part name="P+2" library="supply1" deviceset="+5V" device=""/>
 <part name="GND2" library="supply1" deviceset="GND" device=""/>
+<part name="IN+1" library="pinhead" deviceset="PINHD-1X1" device=""/>
+<part name="IN-1" library="pinhead" deviceset="PINHD-1X1" device=""/>
 </parts>
 <sheets>
@@
 <instance part="P+2" gate="1" x="48.26" y="73.66"/>
 <instance part="GND2" gate="1" x="40.64" y="33.02"/>
+<instance part="IN+1" gate="G$1" x="22.86" y="66.04"/>
+<instance part="IN-1" gate="G$1" x="22.86" y="43.18"/>
 </instances>
 <busses>

Commit message: upravy desky
Parts:
- added IN+2, IN+3, IN+4, IN+5: (no value), pinhead:PINHD-1X1
- added SL1: (no value), con-amp-quick:M05
Connections:
- removed net +5V: JP1.1, OUT+.1
- new net N$8: JP1.3, SL1.2
- new net N$9: JP1.4, SL1.1
- net +3V3: now also IN+3.1, OUT+.1, SL1.5
- net GND: now also IN+4.1, SL1.4
- net N$6: now also IN+2.1
- net N$7: now also IN+5.1
Changed lines of the file:
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@@
 <part name="JP3" library="pinhead" deviceset="PINHD-1X8" device=""/>
 <part name="+3V1" library="supply1" deviceset="+3V3" device=""/>
-<part name="P+1" library="supply1" deviceset="+5V" device=""/>
 <part name="GND1" library="supply1" deviceset="GND" device=""/>
 <part name="DS18B20" library="pinhead" deviceset="PINHD-1X3" device=""/>
@@
 <part name="BAT-1" library="pinhead" deviceset="PINHD-1X1" device=""/>
 <part name="BAT+1" library="pinhead" deviceset="PINHD-1X1" device=""/>
-<part name="P+2" library="supply1" deviceset="+5V" device=""/>
 <part name="GND2" library="supply1" deviceset="GND" device=""/>
 <part name="IN+1" library="pinhead" deviceset="PINHD-1X1" device=""/>
 <part name="IN-1" library="pinhead" deviceset="PINHD-1X1" device=""/>
+<part name="IN+2" library="pinhead" deviceset="PINHD-1X1" device=""/>
+<part name="IN+3" library="pinhead" deviceset="PINHD-1X1" device=""/>
+<part name="SL1" library="con-amp-quick" deviceset="M05" device=""/>
+<part name="IN+4" library="pinhead" deviceset="PINHD-1X1" device=""/>
+<part name="IN+5" library="pinhead" deviceset="PINHD-1X1" device=""/>
 </parts>
 <sheets>
@@
 <instance part="JP3" gate="A" x="78.74" y="55.88" rot="R270"/>
 <instance part="+3V1" gate="G$1" x="71.12" y="73.66"/>
-<instance part="P+1" gate="1" x="71.12" y="35.56" rot="R180"/>
-<instance part="GND1" gate="1" x="73.66" y="25.4"/>
+<instance part="GND1" gate="1" x="66.04" y="38.1"/>
 <instance part="DS18B20" gate="A" x="109.22" y="78.74" rot="R90"/>
 <instance part="R1" gate="G$1" x="104.14" y="60.96" rot="R180"/>
@@
 <instance part="BAT-1" gate="G$1" x="58.42" y="50.8"/>
 <instance part="BAT+1" gate="G$1" x="58.42" y="58.42"/>
-<instance part="P+2" gate="1" x="48.26" y="73.66"/>
 <instance part="GND2" gate="1" x="40.64" y="33.02"/>
 <instance part="IN+1" gate="G$1" x="22.86" y="66.04"/>
 <instance part="IN-1" gate="G$1" x="22.86" y="43.18"/>
+<instance part="IN+2" gate="G$1" x="53.34" y="78.74" rot="R180"/>
+<instance part="IN+3" gate="G$1" x="43.18" y="78.74"/>
+<instance part="SL1" gate="G$1" x="86.36" y="22.86" rot="R90"/>
+<instance part="IN+4" gate="G$1" x="43.18" y="22.86"/>
+<instance part="IN+5" gate="G$1" x="53.34" y="22.86" rot="R180"/>
 </instances>
 <busses>
@@
 <wire x1="99.06" y1="60.96" x2="99.06" y2="68.58" width="0.1524" layer="91"/>
 <junction x="99.06" y="68.58"/>
-</segment>
-</net>
-<net name="+5V" class="0">
-<segment>
-<pinref part="JP1" gate="A" pin="1"/>
-<pinref part="P+1" gate="1" pin="+5V"/>
-<wire x1="71.12" y1="48.26" x2="71.12" y2="38.1" width="0.1524" layer="91"/>
-</segment>
-<segment>
+<pinref part="SL1" gate="G$1" pin="5"/>
+<wire x1="81.28" y1="30.48" x2="81.28" y2="33.02" width="0.1524" layer="91"/>
+<wire x1="81.28" y1="33.02" x2="99.06" y2="33.02" width="0.1524" layer="91"/>
+<wire x1="99.06" y1="33.02" x2="99.06" y2="60.96" width="0.1524" layer="91"/>
+<junction x="99.06" y="60.96"/>
 <pinref part="OUT+" gate="G$1" pin="1"/>
-<wire x1="40.64" y1="66.04" x2="40.64" y2="71.12" width="0.1524" layer="91"/>
-<pinref part="P+2" gate="1" pin="+5V"/>
-<wire x1="40.64" y1="71.12" x2="48.26" y2="71.12" width="0.1524" layer="91"/>
+<wire x1="40.64" y1="66.04" x2="40.64" y2="68.58" width="0.1524" layer="91"/>
+<pinref part="IN+3" gate="G$1" pin="1"/>
+<wire x1="40.64" y1="68.58" x2="40.64" y2="78.74" width="0.1524" layer="91"/>
+<wire x1="71.12" y1="68.58" x2="40.64" y2="68.58" width="0.1524" layer="91"/>
+<junction x="40.64" y="68.58"/>
 </segment>
 </net>
@@
 <pinref part="GND1" gate="1" pin="GND"/>
 <wire x1="73.66" y1="48.26" x2="73.66" y2="40.64" width="0.1524" layer="91"/>
-<wire x1="73.66" y1="40.64" x2="73.66" y2="27.94" width="0.1524" layer="91"/>
-<wire x1="73.66" y1="40.64" x2="111.76" y2="40.64" width="0.1524" layer="91"/>
+<wire x1="73.66" y1="40.64" x2="66.04" y2="40.64" width="0.1524" layer="91"/>
+<wire x1="73.66" y1="40.64" x2="83.82" y2="40.64" width="0.1524" layer="91"/>
 <junction x="73.66" y="40.64"/>
 <pinref part="DS18B20" gate="A" pin="3"/>
+<wire x1="83.82" y1="40.64" x2="111.76" y2="40.64" width="0.1524" layer="91"/>
 <wire x1="111.76" y1="76.2" x2="111.76" y2="40.64" width="0.1524" layer="91"/>
+<pinref part="SL1" gate="G$1" pin="4"/>
+<wire x1="83.82" y1="30.48" x2="83.82" y2="40.64" width="0.1524" layer="91"/>
+<junction x="83.82" y="40.64"/>
 </segment>
 <segment>
@@
 <pinref part="OUT-" gate="G$1" pin="1"/>
 <wire x1="40.64" y1="35.56" x2="40.64" y2="43.18" width="0.1524" layer="91"/>
+<wire x1="40.64" y1="43.18" x2="30.48" y2="43.18" width="0.1524" layer="91"/>
+<wire x1="30.48" y1="43.18" x2="30.48" y2="22.86" width="0.1524" layer="91"/>
+<junction x="40.64" y="43.18"/>
+<pinref part="IN+4" gate="G$1" pin="1"/>
+<wire x1="30.48" y1="22.86" x2="40.64" y2="22.86" width="0.1524" layer="91"/>
 </segment>
 </net>
@@
 </segment>
 </net>
-<net name="N$6" class="0">
-<segment>
-<pinref part="BAT+1" gate="G$1" pin="1"/>
-<pinref part="BAT+" gate="G$1" pin="1"/>
-<wire x1="55.88" y1="58.42" x2="40.64" y2="58.42" width="0.1524" layer="91"/>
-</segment>
-</net>
 <net name="N$7" class="0">
 <segment>
@@
 <pinref part="BAT-" gate="G$1" pin="1"/>
 <wire x1="55.88" y1="50.8" x2="40.64" y2="50.8" width="0.1524" layer="91"/>
+<pinref part="IN+5" gate="G$1" pin="1"/>
+<wire x1="55.88" y1="50.8" x2="55.88" y2="22.86" width="0.1524" layer="91"/>
+<junction x="55.88" y="50.8"/>
 </segment>
 </net>
+<net name="N$8" class="0">
+<segment>
+<pinref part="JP1" gate="A" pin="3"/>
+<wire x1="76.2" y1="48.26" x2="76.2" y2="35.56" width="0.1524" layer="91"/>
+<pinref part="SL1" gate="G$1" pin="2"/>
+<wire x1="76.2" y1="35.56" x2="88.9" y2="35.56" width="0.1524" layer="91"/>
+<wire x1="88.9" y1="35.56" x2="88.9" y2="30.48" width="0.1524" layer="91"/>
+</segment>
+</net>
+<net name="N$9" class="0">
+<segment>
+<pinref part="JP1" gate="A" pin="4"/>
+<wire x1="78.74" y1="48.26" x2="78.74" y2="38.1" width="0.1524" layer="91"/>
+<pinref part="SL1" gate="G$1" pin="1"/>
+<wire x1="78.74" y1="38.1" x2="91.44" y2="38.1" width="0.1524" layer="91"/>
+<wire x1="91.44" y1="38.1" x2="91.44" y2="30.48" width="0.1524" layer="91"/>
+</segment>
+</net>
+<net name="N$6" class="0">
+<segment>
+<pinref part="BAT+" gate="G$1" pin="1"/>
+<pinref part="BAT+1" gate="G$1" pin="1"/>
+<junction x="55.88" y="58.42"/>
+<pinref part="IN+2" gate="G$1" pin="1"/>
+<wire x1="55.88" y1="78.74" x2="55.88" y2="58.42" width="0.1524" layer="91"/>
+<wire x1="55.88" y1="58.42" x2="40.64" y2="58.42" width="0.1524" layer="91"/>
+</segment>
+</net>
