File: iSpindel/deska.brd (EAGLE design)
At the start: 49.2 x 36.8 mm, 14 parts

Commit message: zmeny desky
Parts:
- moved DS18B20 34.3 mm to (3.81, 19.1)
- moved R1 23.2 mm to (11.4, 19.1), turned to 0 degrees
- moved R3 13.4 mm to (38.1, 25.4), turned to 180 degrees
- moved R2 7.73 mm to (16.5, 26.6)
- moved BAT-1 1.27 mm to (44.5, 21.6)
Connections:
- net +5V: now also OUT+.1
- net GND: now also OUT-.1
Routing:
- net GND: track 0.00 -> 39.5 mm
- net +3V3: track 0.00 -> 23.9 mm
- net +5V: track 0.00 -> 20.8 mm
- net N$4: track 0.00 -> 19.3 mm
- net N$7: track 0.00 -> 14.1 mm
- net N$6: track 0.00 -> 14.0 mm
- net N$1: track 0.00 -> 10.7 mm
- net N$3: track 0.00 -> 8.11 mm
- net N$2: track 0.00 -> 3.81 mm
Other:
- board size 49.2 x 36.8 mm -> 49.2 x 29.2 mm
Changed lines of the file:
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@@
 <setting verticaltext="up"/>
 </settings>
-<grid distance="100" unitdist="mil" unit="mil" style="lines" multiple="1" display="no" altdistance="0.025" altunitdist="inch" altunit="mm"/>
+<grid distance="50" unitdist="mil" unit="mil" style="lines" multiple="1" display="no" altdistance="984.251969" altunitdist="mil" altunit="mil"/>
 <layers>
 <layer number="1" name="Top" color="4" fill="1" visible="yes" active="yes"/>
@@
 <board>
 <plain>
-<wire x1="0" y1="0" x2="49.2" y2="0" width="0" layer="20"/>
-<wire x1="49.2" y1="0" x2="49.2" y2="36.82" width="0" layer="20"/>
-<wire x1="49.2" y1="36.82" x2="0" y2="36.82" width="0" layer="20"/>
-<wire x1="0" y1="36.82" x2="0" y2="0" width="0" layer="20"/>
-<dimension x1="15.24" y1="7.62" x2="15.24" y2="30.48" x3="-2.54" y3="19.05" textsize="1.778" layer="16"/>
-<dimension x1="13.97" y1="11.43" x2="13.97" y2="24.13" x3="5.08" y3="17.78" textsize="1.778" layer="16"/>
-<dimension x1="8.89" y1="11.43" x2="30.48" y2="11.43" x3="19.685" y3="2.54" textsize="1.778" layer="16"/>
-<dimension x1="30.48" y1="21.59" x2="30.48" y2="13.97" x3="25.4" y3="17.78" textsize="1.778" layer="16"/>
+<wire x1="0" y1="5.08" x2="49.2" y2="5.08" width="0" layer="20"/>
+<wire x1="49.2" y1="5.08" x2="49.2" y2="34.28" width="0" layer="20"/>
+<wire x1="49.2" y1="34.28" x2="0" y2="34.28" width="0" layer="20"/>
+<wire x1="0" y1="34.28" x2="0" y2="5.08" width="0" layer="20"/>
 </plain>
 <attributes>
@@
 <autorouter>
 <pass name="Default">
-<param name="RoutingGrid" value="50mil"/>
-<param name="AutoGrid" value="1"/>
+<param name="RoutingGrid" value="12.5mil"/>
+<param name="AutoGrid" value="0"/>
 <param name="Efforts" value="0"/>
 <param name="TopRouterVariant" value="1"/>
 <param name="tpViaShape" value="round"/>
-<param name="PrefDir.1" value="a"/>
+<param name="PrefDir.1" value="-"/>
 <param name="PrefDir.2" value="0"/>
 <param name="PrefDir.3" value="0"/>
@@
 <param name="PrefDir.14" value="0"/>
 <param name="PrefDir.15" value="0"/>
-<param name="PrefDir.16" value="a"/>
+<param name="PrefDir.16" value="|"/>
 <param name="cfVia" value="8"/>
 <param name="cfNonPref" value="5"/>
@@
 <element name="BAT+" library="pinhead" package="1X01" value="" x="30.48" y="13.97"/>
 <element name="BAT-" library="pinhead" package="1X01" value="" x="30.48" y="21.59"/>
-<element name="DS18B20" library="pinhead" package="1X03" value="" x="38.1" y="19.05" rot="R270"/>
+<element name="DS18B20" library="pinhead" package="1X03" value="" x="3.81" y="19.05" rot="R270"/>
 <element name="IN+" library="pinhead" package="1X01" value="" x="8.89" y="11.43"/>
 <element name="IN-" library="pinhead" package="1X01" value="" x="8.89" y="24.13"/>
@@
 <element name="OUT+" library="pinhead" package="1X01" value="" x="30.48" y="11.43"/>
 <element name="OUT-" library="pinhead" package="1X01" value="" x="30.48" y="24.13"/>
-<element name="R1" library="rcl" package="0204/7" value="4k7" x="34.29" y="22.86" rot="R90"/>
-<element name="R2" library="rcl" package="0204/7" value="230k" x="15.24" y="34.25"/>
-<element name="R3" library="rcl" package="0204/7" value="470" x="27.94" y="34.25"/>
-<element name="BAT-1" library="pinhead" package="1X01" value="" x="44.45" y="22.86"/>
+<element name="R1" library="rcl" package="0204/7" value="4k7" x="11.43" y="19.05"/>
+<element name="R2" library="rcl" package="0204/7" value="230k" x="16.51" y="26.63"/>
+<element name="R3" library="rcl" package="0204/7" value="470" x="38.1" y="25.44" rot="R180"/>
+<element name="BAT-1" library="pinhead" package="1X01" value="" x="44.45" y="21.59"/>
 <element name="BAT+1" library="pinhead" package="1X01" value="" x="44.45" y="13.97"/>
 </elements>
@@
 <contactref element="R2" pad="1"/>
 <contactref element="R1" pad="2"/>
-<wire x1="12.7" y1="30.48" x2="11.43" y2="34.25" width="0" layer="19" extent="1-1"/>
-<wire x1="38.1" y1="21.59" x2="12.7" y2="30.48" width="0" layer="19" extent="1-1"/>
-<wire x1="34.29" y1="26.67" x2="38.1" y2="21.59" width="0" layer="19" extent="1-1"/>
+<wire x1="15.0876" y1="24.2316" x2="15.0876" y2="21.717" width="0.6096" layer="1"/>
+<wire x1="15.0876" y1="21.717" x2="15.0876" y2="19.2024" width="0.6096" layer="1"/>
+<wire x1="12.8016" y1="26.5176" x2="15.0876" y2="24.2316" width="0.6096" layer="1"/>
+<wire x1="15.0876" y1="19.2024" x2="15.24" y2="19.05" width="0.6096" layer="1"/>
+<wire x1="12.8016" y1="26.5176" x2="12.7" y2="26.63" width="0.254" layer="1"/>
+<wire x1="15.0876" y1="21.717" x2="3.8862" y2="21.717" width="0.6096" layer="1"/>
+<wire x1="3.8862" y1="21.717" x2="3.81" y2="21.59" width="0.254" layer="1"/>
+<wire x1="12.8016" y1="26.7462" x2="12.8016" y2="30.4038" width="0.6096" layer="1"/>
+<wire x1="12.8016" y1="30.4038" x2="12.7" y2="30.48" width="0.254" layer="1"/>
+<wire x1="12.8016" y1="26.7462" x2="12.7" y2="26.63" width="0.254" layer="1"/>
 </signal>
 <signal name="+5V">
 <contactref element="JP1" pad="1"/>
+<contactref element="OUT+" pad="1"/>
+<wire x1="30.48" y1="11.43" x2="13.97" y2="11.43" width="0.6096" layer="16"/>
+<wire x1="13.97" y1="11.43" x2="12.7" y2="10.16" width="0.6096" layer="16"/>
+<wire x1="12.7" y1="10.16" x2="12.7" y2="7.62" width="0.6096" layer="16"/>
 </signal>
 <signal name="GND">
 <contactref element="JP1" pad="2"/>
 <contactref element="DS18B20" pad="3"/>
-<wire x1="15.24" y1="7.62" x2="38.1" y2="16.51" width="0" layer="19" extent="1-1"/>
+<wire x1="15.3162" y1="7.7724" x2="15.24" y2="7.62" width="0.254" layer="1"/>
+<wire x1="3.8862" y1="16.4592" x2="3.81" y2="16.51" width="0.254" layer="1"/>
+<contactref element="OUT-" pad="1"/>
+<wire x1="30.4038" y1="24.003" x2="30.48" y2="24.13" width="0.254" layer="1"/>
+<wire x1="14.6304" y1="8.2296" x2="15.24" y2="7.62" width="0.254" layer="1"/>
+<wire x1="3.8862" y1="16.4592" x2="14.0208" y2="16.4592" width="0.6096" layer="1"/>
+<wire x1="14.0208" y1="16.4592" x2="15.24" y2="15.24" width="0.6096" layer="1"/>
+<wire x1="15.24" y1="15.24" x2="15.24" y2="7.62" width="0.6096" layer="1"/>
+<wire x1="30.4038" y1="24.003" x2="29.083" y2="24.003" width="0.6096" layer="1"/>
+<wire x1="29.083" y1="24.003" x2="20.32" y2="15.24" width="0.6096" layer="1"/>
+<wire x1="20.32" y1="15.24" x2="15.24" y2="15.24" width="0.6096" layer="1"/>
 </signal>
 <signal name="N$2">
 <contactref element="DS18B20" pad="2"/>
 <contactref element="R1" pad="1"/>
-<wire x1="38.1" y1="19.05" x2="34.29" y2="19.05" width="0" layer="19" extent="1-1"/>
+<wire x1="7.62" y1="19.05" x2="3.81" y2="19.05" width="0.6096" layer="1"/>
 </signal>
 <signal name="N$1">
 <contactref element="JP3" pad="2"/>
 <contactref element="R2" pad="2"/>
-<wire x1="19.05" y1="34.25" x2="27.94" y2="30.48" width="0" layer="19" extent="1-1"/>
+<wire x1="20.32" y1="26.63" x2="26.63" y2="26.63" width="0.6096" layer="1"/>
+<wire x1="26.63" y1="26.63" x2="27.94" y2="27.94" width="0.6096" layer="1"/>
+<wire x1="27.94" y1="27.94" x2="27.94" y2="30.48" width="0.6096" layer="1"/>
 </signal>
 <signal name="N$3">
 <contactref element="JP3" pad="1"/>
 <contactref element="R3" pad="2"/>
-<wire x1="31.75" y1="34.25" x2="30.48" y2="30.48" width="0" layer="19" extent="1-1"/>
+<wire x1="30.48" y1="30.48" x2="33.02" y2="30.48" width="0.6096" layer="1"/>
+<wire x1="33.02" y1="30.48" x2="34.29" y2="29.21" width="0.6096" layer="1"/>
+<wire x1="34.29" y1="29.21" x2="34.29" y2="25.44" width="0.6096" layer="1"/>
 </signal>
 <signal name="N$4">
 <contactref element="JP3" pad="3"/>
 <contactref element="R3" pad="1"/>
-<wire x1="24.13" y1="34.25" x2="25.4" y2="30.48" width="0" layer="19" extent="1-1"/>
+<wire x1="25.4" y1="30.48" x2="25.4" y2="29.21" width="0.6096" layer="16"/>
+<wire x1="25.4" y1="29.21" x2="27.94" y2="26.67" width="0.6096" layer="16"/>
+<wire x1="27.94" y1="26.67" x2="40.68" y2="26.67" width="0.6096" layer="16"/>
+<wire x1="40.68" y1="26.67" x2="41.91" y2="25.44" width="0.6096" layer="16"/>
 </signal>
 <signal name="N$6">
 <contactref element="BAT+1" pad="1"/>
 <contactref element="BAT+" pad="1"/>
-<wire x1="30.48" y1="13.97" x2="44.45" y2="13.97" width="0" layer="19" extent="1-1"/>
+<wire x1="44.3484" y1="13.9446" x2="30.6324" y2="13.9446" width="0.8128" layer="1"/>
+<wire x1="30.6324" y1="13.9446" x2="30.48" y2="13.97" width="0.254" layer="1"/>
+<wire x1="44.3484" y1="13.9446" x2="44.45" y2="13.97" width="0.254" layer="1"/>
 </signal>
 <signal name="N$7">
 <contactref element="BAT-1" pad="1"/>
 <contactref element="BAT-" pad="1"/>
-<wire x1="44.45" y1="22.86" x2="30.48" y2="21.59" width="0" layer="19" extent="1-1"/>
+<wire x1="44.3484" y1="21.717" x2="30.6324" y2="21.717" width="0.8128" layer="1"/>
+<wire x1="30.6324" y1="21.717" x2="30.48" y2="21.59" width="0.254" layer="1"/>
+<wire x1="44.3484" y1="21.717" x2="44.45" y2="21.59" width="0.254" layer="1"/>
 </signal>
 </signals>

Commit message: deska
Parts:
- added IN+1, IN-1: (no value), pinhead:1X01
- moved IN- 4.02 mm to (12.7, 25.4)
- moved IN+ 3.81 mm to (12.7, 11.4)
- moved R2 3.81 mm to (20.3, 26.6)
- moved OUT- 1.27 mm to (30.5, 25.4)
- moved BAT- 0.64 mm to (30.5, 22.2)
- moved BAT-1 0.64 mm to (44.5, 22.2)
- moved BAT+ 0.63 mm to (30.5, 14.6)
- moved BAT+1 0.63 mm to (44.5, 14.6)
Routing:
- net +3V3: track 23.9 -> 30.5 mm
- net N$1: track 10.7 -> 6.89 mm
- net +5V: track 20.8 -> 20.1 mm
Changed lines of the file:
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@@
 <setting verticaltext="up"/>
 </settings>
-<grid distance="50" unitdist="mil" unit="mil" style="lines" multiple="1" display="no" altdistance="984.251969" altunitdist="mil" altunit="mil"/>
+<grid distance="25" unitdist="mil" unit="mil" style="lines" multiple="1" display="no" altdistance="984.251969" altunitdist="mil" altunit="mil"/>
 <layers>
 <layer number="1" name="Top" color="4" fill="1" visible="yes" active="yes"/>
@@
 <board>
 <plain>
-<wire x1="0" y1="5.08" x2="49.2" y2="5.08" width="0" layer="20"/>
-<wire x1="49.2" y1="5.08" x2="49.2" y2="34.28" width="0" layer="20"/>
-<wire x1="49.2" y1="34.28" x2="0" y2="34.28" width="0" layer="20"/>
-<wire x1="0" y1="34.28" x2="0" y2="5.08" width="0" layer="20"/>
+<wire x1="0" y1="4.445" x2="49.2" y2="4.445" width="0" layer="20"/>
+<wire x1="49.2" y1="4.445" x2="49.2" y2="33.645" width="0" layer="20"/>
+<wire x1="49.2" y1="33.645" x2="0" y2="33.645" width="0" layer="20"/>
+<wire x1="0" y1="33.645" x2="0" y2="4.445" width="0" layer="20"/>
 </plain>
 <attributes>
@@
 </autorouter>
 <elements>
-<element name="BAT+" library="pinhead" package="1X01" value="" x="30.48" y="13.97"/>
-<element name="BAT-" library="pinhead" package="1X01" value="" x="30.48" y="21.59"/>
+<element name="BAT+" library="pinhead" package="1X01" value="" x="30.48" y="14.605"/>
+<element name="BAT-" library="pinhead" package="1X01" value="" x="30.48" y="22.225"/>
 <element name="DS18B20" library="pinhead" package="1X03" value="" x="3.81" y="19.05" rot="R270"/>
-<element name="IN+" library="pinhead" package="1X01" value="" x="8.89" y="11.43"/>
-<element name="IN-" library="pinhead" package="1X01" value="" x="8.89" y="24.13"/>
+<element name="IN+" library="pinhead" package="1X01" value="" x="12.7" y="11.43"/>
+<element name="IN-" library="pinhead" package="1X01" value="" x="12.7" y="25.4"/>
 <element name="JP1" library="pinhead" package="1X08" value="" x="21.59" y="7.62"/>
 <element name="JP3" library="pinhead" package="1X08" value="" x="21.59" y="30.48" rot="R180"/>
 <element name="OUT+" library="pinhead" package="1X01" value="" x="30.48" y="11.43"/>
-<element name="OUT-" library="pinhead" package="1X01" value="" x="30.48" y="24.13"/>
+<element name="OUT-" library="pinhead" package="1X01" value="" x="30.48" y="25.4"/>
 <element name="R1" library="rcl" package="0204/7" value="4k7" x="11.43" y="19.05"/>
-<element name="R2" library="rcl" package="0204/7" value="230k" x="16.51" y="26.63"/>
+<element name="R2" library="rcl" package="0204/7" value="230k" x="20.32" y="26.63"/>
 <element name="R3" library="rcl" package="0204/7" value="470" x="38.1" y="25.44" rot="R180"/>
-<element name="BAT-1" library="pinhead" package="1X01" value="" x="44.45" y="21.59"/>
-<element name="BAT+1" library="pinhead" package="1X01" value="" x="44.45" y="13.97"/>
+<element name="BAT-1" library="pinhead" package="1X01" value="" x="44.45" y="22.225"/>
+<element name="BAT+1" library="pinhead" package="1X01" value="" x="44.45" y="14.605"/>
+<element name="IN+1" library="pinhead" package="1X01" value="" x="8.89" y="11.43"/>
+<element name="IN-1" library="pinhead" package="1X01" value="" x="8.89" y="25.4"/>
 </elements>
 <signals>
@@
 <contactref element="R2" pad="1"/>
 <contactref element="R1" pad="2"/>
-<wire x1="15.0876" y1="24.2316" x2="15.0876" y2="21.717" width="0.6096" layer="1"/>
-<wire x1="15.0876" y1="21.717" x2="15.0876" y2="19.2024" width="0.6096" layer="1"/>
-<wire x1="12.8016" y1="26.5176" x2="15.0876" y2="24.2316" width="0.6096" layer="1"/>
-<wire x1="15.0876" y1="19.2024" x2="15.24" y2="19.05" width="0.6096" layer="1"/>
-<wire x1="12.8016" y1="26.5176" x2="12.7" y2="26.63" width="0.254" layer="1"/>
-<wire x1="15.0876" y1="21.717" x2="3.8862" y2="21.717" width="0.6096" layer="1"/>
-<wire x1="3.8862" y1="21.717" x2="3.81" y2="21.59" width="0.254" layer="1"/>
-<wire x1="12.8016" y1="26.7462" x2="12.8016" y2="30.4038" width="0.6096" layer="1"/>
-<wire x1="12.8016" y1="30.4038" x2="12.7" y2="30.48" width="0.254" layer="1"/>
-<wire x1="12.8016" y1="26.7462" x2="12.7" y2="26.63" width="0.254" layer="1"/>
+<wire x1="12.7" y1="30.48" x2="12.7" y2="29.21" width="0.6096" layer="1"/>
+<wire x1="12.7" y1="29.21" x2="15.24" y2="26.67" width="0.6096" layer="1"/>
+<wire x1="15.24" y1="26.67" x2="16.47" y2="26.67" width="0.6096" layer="1"/>
+<wire x1="16.47" y1="26.67" x2="16.51" y2="26.63" width="0.6096" layer="1"/>
+<wire x1="15.24" y1="19.05" x2="16.51" y2="20.32" width="0.6096" layer="1"/>
+<wire x1="16.51" y1="20.32" x2="16.51" y2="26.63" width="0.6096" layer="1"/>
+<wire x1="3.81" y1="21.59" x2="5.08" y2="21.59" width="0.6096" layer="1"/>
+<wire x1="12.7" y1="29.21" x2="6.35" y2="29.21" width="0.6096" layer="1"/>
+<wire x1="6.35" y1="29.21" x2="3.81" y2="26.67" width="0.6096" layer="1"/>
+<wire x1="3.81" y1="26.67" x2="3.81" y2="21.59" width="0.6096" layer="1"/>
 </signal>
 <signal name="+5V">
 <contactref element="JP1" pad="1"/>
 <contactref element="OUT+" pad="1"/>
-<wire x1="30.48" y1="11.43" x2="13.97" y2="11.43" width="0.6096" layer="16"/>
-<wire x1="13.97" y1="11.43" x2="12.7" y2="10.16" width="0.6096" layer="16"/>
-<wire x1="12.7" y1="10.16" x2="12.7" y2="7.62" width="0.6096" layer="16"/>
+<wire x1="30.48" y1="11.43" x2="15.24" y2="11.43" width="0.6096" layer="16"/>
+<wire x1="15.24" y1="11.43" x2="12.7" y2="8.89" width="0.6096" layer="16"/>
+<wire x1="12.7" y1="8.89" x2="12.7" y2="7.62" width="0.6096" layer="16"/>
 </signal>
 <signal name="GND">
@@
 <contactref element="DS18B20" pad="3"/>
 <wire x1="15.3162" y1="7.7724" x2="15.24" y2="7.62" width="0.254" layer="1"/>
-<wire x1="3.8862" y1="16.4592" x2="3.81" y2="16.51" width="0.254" layer="1"/>
 <contactref element="OUT-" pad="1"/>
-<wire x1="30.4038" y1="24.003" x2="30.48" y2="24.13" width="0.254" layer="1"/>
 <wire x1="14.6304" y1="8.2296" x2="15.24" y2="7.62" width="0.254" layer="1"/>
-<wire x1="3.8862" y1="16.4592" x2="14.0208" y2="16.4592" width="0.6096" layer="1"/>
-<wire x1="14.0208" y1="16.4592" x2="15.24" y2="15.24" width="0.6096" layer="1"/>
-<wire x1="15.24" y1="15.24" x2="15.24" y2="7.62" width="0.6096" layer="1"/>
-<wire x1="30.4038" y1="24.003" x2="29.083" y2="24.003" width="0.6096" layer="1"/>
-<wire x1="29.083" y1="24.003" x2="20.32" y2="15.24" width="0.6096" layer="1"/>
-<wire x1="20.32" y1="15.24" x2="15.24" y2="15.24" width="0.6096" layer="1"/>
+<wire x1="3.81" y1="16.51" x2="12.7" y2="16.51" width="0.6096" layer="1"/>
+<wire x1="12.7" y1="16.51" x2="15.24" y2="13.97" width="0.6096" layer="1"/>
+<wire x1="15.24" y1="13.97" x2="15.24" y2="7.62" width="0.6096" layer="1"/>
+<wire x1="30.48" y1="25.4" x2="26.67" y2="25.4" width="0.6096" layer="1"/>
+<wire x1="26.67" y1="25.4" x2="15.24" y2="13.97" width="0.6096" layer="1"/>
 </signal>
 <signal name="N$2">
@@
 <contactref element="JP3" pad="2"/>
 <contactref element="R2" pad="2"/>
-<wire x1="20.32" y1="26.63" x2="26.63" y2="26.63" width="0.6096" layer="1"/>
+<wire x1="24.13" y1="26.63" x2="26.63" y2="26.63" width="0.6096" layer="1"/>
 <wire x1="26.63" y1="26.63" x2="27.94" y2="27.94" width="0.6096" layer="1"/>
 <wire x1="27.94" y1="27.94" x2="27.94" y2="30.48" width="0.6096" layer="1"/>
@@
 <contactref element="BAT+1" pad="1"/>
 <contactref element="BAT+" pad="1"/>
-<wire x1="44.3484" y1="13.9446" x2="30.6324" y2="13.9446" width="0.8128" layer="1"/>
-<wire x1="30.6324" y1="13.9446" x2="30.48" y2="13.97" width="0.254" layer="1"/>
-<wire x1="44.3484" y1="13.9446" x2="44.45" y2="13.97" width="0.254" layer="1"/>
+<wire x1="30.48" y1="14.605" x2="44.45" y2="14.605" width="0.6096" layer="1"/>
 </signal>
 <signal name="N$7">
 <contactref element="BAT-1" pad="1"/>
 <contactref element="BAT-" pad="1"/>
-<wire x1="44.3484" y1="21.717" x2="30.6324" y2="21.717" width="0.8128" layer="1"/>
-<wire x1="30.6324" y1="21.717" x2="30.48" y2="21.59" width="0.254" layer="1"/>
-<wire x1="44.3484" y1="21.717" x2="44.45" y2="21.59" width="0.254" layer="1"/>
+<wire x1="30.48" y1="22.225" x2="44.45" y2="22.225" width="0.6096" layer="1"/>
 </signal>
 </signals>

Commit message: upravy desky
Parts:
- added IN+2, IN+3, IN+4, IN+5: (no value), pinhead:1X01
- added SL1: (no value), con-amp-quick:05P
- moved R3 5.24 mm to (36.8, 30.5)
Connections:
- removed net +5V: JP1.1, OUT+.1
- new net N$8: JP1.3, SL1.2
- new net N$9: JP1.4, SL1.1
- net +3V3: now also IN+3.1, OUT+.1, SL1.5
- net GND: now also IN+4.1, SL1.4
- net N$6: now also IN+2.1
- net N$7: now also IN+5.1
Routing:
- net GND: track 39.8 -> 92.3 mm
- net +3V3: track 30.5 -> 65.3 mm, vias 0 -> 1
- net +5V: track 20.1 -> 0.00 mm
- net N$8: track 0.00 -> 11.2 mm
- net N$9: track 0.00 -> 10.8 mm
- net N$3: track 8.11 -> 2.58 mm
- net N$4: track 19.3 -> 17.9 mm
- net N$1: track 6.89 -> 6.15 mm

Commit message: kalib
Parts:
- moved R3 1.91 mm to (36.8, 28.6)
Routing:
- net N$4: track 17.9 -> 19.8 mm
- net N$3: track 2.58 -> 3.31 mm
Changed lines of the file:
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@@
 <element name="R1" library="rcl" package="0204/7" value="4k7" x="11.43" y="19.05"/>
 <element name="R2" library="rcl" package="0204/7" value="230k" x="20.32" y="26.63"/>
-<element name="R3" library="rcl" package="0204/7" value="470" x="36.83" y="30.52" rot="R180"/>
+<element name="R3" library="rcl" package="0204/7" value="470" x="36.83" y="28.615" rot="R180"/>
 <element name="BAT-1" library="pinhead" package="1X01" value="" x="44.45" y="22.225"/>
 <element name="BAT+1" library="pinhead" package="1X01" value="" x="44.45" y="14.605"/>
@@
 <contactref element="JP3" pad="1"/>
 <contactref element="R3" pad="2"/>
-<wire x1="30.48" y1="30.48" x2="33.02" y2="30.48" width="0.6096" layer="16"/>
-<wire x1="33.02" y1="30.48" x2="33.02" y2="30.52" width="0.4064" layer="16"/>
+<wire x1="30.48" y1="30.48" x2="31.155" y2="30.48" width="0.4064" layer="16"/>
+<wire x1="31.155" y1="30.48" x2="33.02" y2="28.615" width="0.4064" layer="16"/>
 </signal>
 <signal name="N$4">
 <contactref element="JP3" pad="3"/>
 <contactref element="R3" pad="1"/>
-<wire x1="40.64" y1="30.52" x2="40.64" y2="31.115" width="0.4064" layer="16"/>
+<wire x1="40.64" y1="28.615" x2="40.64" y2="31.115" width="0.4064" layer="16"/>
 <wire x1="40.64" y1="31.115" x2="39.37" y2="32.385" width="0.4064" layer="16"/>
 <wire x1="39.37" y1="32.385" x2="26.035" y2="32.385" width="0.4064" layer="16"/>
